Commit message: [orbbec astra camera urdf +]

File: week2_slam/install/vicpinky_description/share/vicpinky_description/urdf/camera.xacro (robot description, xacro)
@@ -2,22 +2,24 @@
 <robot xmlns:xacro="http://www.ros.org/wiki/xacro">
     <xacro:arg name="namespace" default=""/>
-    <xacro:property name="prefix" value="$(arg namespace)"/>
-    <gazebo reference="${prefix}camera_link">
-      <sensor name="camera" type="rgbd_camera">
-        <update_rate>30.0</update_rate>
-        <topic>/astra</topic>
-        <camera name="astra">
-          <horizontal_fov>1.047</horizontal_fov>
-          <image>
-            <width>640</width>
-            <height>480</height>
-            <format>R8G8B8</format>
-          </image>
-          <clip>
-            <near>0.6</near>
-            <far>8.0</far>
-          </clip>
-        </camera>
-        </sensor>
-    </gazebo>
+    <property name="prefix" value="$(arg namespace)"/>
+  <gazebo reference="${prefix}camera_link">
+    <sensor name="rgbd_camera" type="rgbd_camera">
+      <camera>
+        <horizontal_fov>1.047</horizontal_fov>
+        <image>
+          <width>640</width>
+          <height>480</height>
+        </image>
+        <clip>
+          <near>0.6</near>
+          <far>8.0</far>
+        </clip>
+      </camera>
+      <always_on>1</always_on>
+      <update_rate>30</update_rate>
+      <visualize>true</visualize>
+      <topic>astra</topic>
+      <gz_frame_id>${prefix}camera_link</gz_frame_id>
+    </sensor>
+  </gazebo>
 </robot>

File: week2_slam/install/vicpinky_description/share/vicpinky_description/urdf/robot_core.xacro (robot description, xacro)
@@ -260,5 +260,5 @@
       <parent link="${prefix}camera_mount"/>
       <child link="${prefix}camera_link"/>
-      <origin xyz="0.035 0.015 0.008" rpy="0 0 0"/>
+      <origin xyz="0.015 0.015 0.008" rpy="0 0 0"/>
     </joint>
 </robot>
